File: Track-Cam.sch (EAGLE design)
At the start: 39 parts, among them IC1 STM32F042KT/M, IC2 BD6211F/M, IC3 BD6211F/M, P1 RASPI_BOARD_B+#_HC

Commit message: optimize wiring
Parts:
- removed U$1: PRODUCT-LOGO-TRACKCAM, logo:PRODUCT-LOGO-TRACKCAM
- removed U$2: OPIOPAN-LOGO, logo:OPIOPAN-LOGO
- added R6, R7, R8, R9: 10K, gen-discrete:RESISTOR-US2012
Connections:
- net GND: now also R6.2, R7.2, R8.2, R9.2
- net MOTOR1_F: now also R6.1
- net MOTOR1_R: now also R7.1
- net MOTOR2_F: now also R8.1
- net MOTOR2_R: now also R9.1
Other:
- moved on the sheet: 1B, 2A, 2B
Changed lines of the file:
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@@
 <part name="GND15" library="supply1" deviceset="GND" device=""/>
 <part name="XMTR" library="connector" deviceset="53047-0310" device=""/>
-<part name="U$1" library="logo" deviceset="PRODUCT-LOGO" device="-TRACKCAM"/>
-<part name="U$2" library="logo" deviceset="OPIOPAN-LOGO" device=""/>
+<part name="R6" library="gen-discrete" deviceset="RESISTOR-US" device="2012" value="10K"/>
+<part name="GND16" library="supply1" deviceset="GND" device=""/>
+<part name="R7" library="gen-discrete" deviceset="RESISTOR-US" device="2012" value="10K"/>
+<part name="GND17" library="supply1" deviceset="GND" device=""/>
+<part name="R8" library="gen-discrete" deviceset="RESISTOR-US" device="2012" value="10K"/>
+<part name="GND18" library="supply1" deviceset="GND" device=""/>
+<part name="R9" library="gen-discrete" deviceset="RESISTOR-US" device="2012" value="10K"/>
+<part name="GND19" library="supply1" deviceset="GND" device=""/>
 </parts>
 <sheets>
@@
 <instance part="POS2" gate="G$1" x="203.2" y="180.34" rot="R180"/>
 <instance part="1A" gate="G$1" x="372.11" y="143.51" rot="R90"/>
-<instance part="1B" gate="G$1" x="379.73" y="143.51" rot="R90"/>
-<instance part="2A" gate="G$1" x="387.35" y="143.51" rot="R90"/>
-<instance part="2B" gate="G$1" x="394.97" y="143.51" rot="R90"/>
+<instance part="1B" gate="G$1" x="384.81" y="143.51" rot="R90"/>
+<instance part="2A" gate="G$1" x="397.51" y="143.51" rot="R90"/>
+<instance part="2B" gate="G$1" x="410.21" y="143.51" rot="R90"/>
 <instance part="R5" gate="G$1" x="349.25" y="156.21" rot="R90"/>
 <instance part="LED3" gate="G$1" x="361.95" y="156.21" rot="R90"/>
 <instance part="GND15" gate="1" x="364.49" y="151.13"/>
 <instance part="XMTR" gate="G$1" x="349.25" y="146.05"/>
-<instance part="U$1" gate="G$1" x="90.17" y="204.47"/>
-<instance part="U$2" gate="G$1" x="120.65" y="203.2"/>
+<instance part="R6" gate="G$1" x="378.46" y="137.16"/>
+<instance part="GND16" gate="1" x="378.46" y="128.27"/>
+<instance part="R7" gate="G$1" x="391.16" y="137.16"/>
+<instance part="GND17" gate="1" x="391.16" y="128.27"/>
+<instance part="R8" gate="G$1" x="403.86" y="137.16"/>
+<instance part="GND18" gate="1" x="403.86" y="128.27"/>
+<instance part="R9" gate="G$1" x="416.56" y="137.16"/>
+<instance part="GND19" gate="1" x="416.56" y="128.27"/>
 </instances>
 <busses>
@@
 <segment>
 <pinref part="1A" gate="G$1" pin="TP"/>
-<wire x1="374.65" y1="143.51" x2="374.65" y2="124.46" width="0.1524" layer="91"/>
+<wire x1="374.65" y1="143.51" x2="374.65" y2="142.24" width="0.1524" layer="91"/>
 <label x="374.65" y="125.73" size="1.778" layer="95" rot="R90"/>
+<pinref part="R6" gate="G$1" pin="1"/>
+<wire x1="374.65" y1="142.24" x2="374.65" y2="124.46" width="0.1524" layer="91"/>
+<wire x1="378.46" y1="142.24" x2="374.65" y2="142.24" width="0.1524" layer="91"/>
+<junction x="374.65" y="142.24"/>
 </segment>
 </net>
@@
 <wire x1="335.28" y1="146.05" x2="335.28" y2="138.43" width="0.1524" layer="91"/>
 </segment>
+<segment>
+<pinref part="R6" gate="G$1" pin="2"/>
+<pinref part="GND16" gate="1" pin="GND"/>
+<wire x1="378.46" y1="130.81" x2="378.46" y2="132.08" width="0.1524" layer="91"/>
+</segment>
+<segment>
+<pinref part="R7" gate="G$1" pin="2"/>
+<pinref part="GND17" gate="1" pin="GND"/>
+<wire x1="391.16" y1="130.81" x2="391.16" y2="132.08" width="0.1524" layer="91"/>
+</segment>
+<segment>
+<pinref part="R8" gate="G$1" pin="2"/>
+<pinref part="GND18" gate="1" pin="GND"/>
+<wire x1="403.86" y1="130.81" x2="403.86" y2="132.08" width="0.1524" layer="91"/>
+</segment>
+<segment>
+<pinref part="R9" gate="G$1" pin="2"/>
+<pinref part="GND19" gate="1" pin="GND"/>
+<wire x1="416.56" y1="130.81" x2="416.56" y2="132.08" width="0.1524" layer="91"/>
+</segment>
 </net>
 <net name="MOTOR2_POS" class="0">
@@
 <segment>
 <pinref part="1B" gate="G$1" pin="TP"/>
-<wire x1="382.27" y1="143.51" x2="382.27" y2="124.46" width="0.1524" layer="91"/>
-<label x="382.27" y="125.73" size="1.778" layer="95" rot="R90"/>
+<wire x1="387.35" y1="143.51" x2="387.35" y2="142.24" width="0.1524" layer="91"/>
+<label x="387.35" y="125.73" size="1.778" layer="95" rot="R90"/>
+<pinref part="R7" gate="G$1" pin="1"/>
+<wire x1="387.35" y1="142.24" x2="387.35" y2="124.46" width="0.1524" layer="91"/>
+<wire x1="391.16" y1="142.24" x2="387.35" y2="142.24" width="0.1524" layer="91"/>
+<junction x="387.35" y="142.24"/>
 </segment>
 </net>
@@
 <segment>
 <pinref part="2A" gate="G$1" pin="TP"/>
-<wire x1="389.89" y1="143.51" x2="389.89" y2="124.46" width="0.1524" layer="91"/>
-<label x="389.89" y="125.73" size="1.778" layer="95" rot="R90"/>
+<wire x1="400.05" y1="143.51" x2="400.05" y2="142.24" width="0.1524" layer="91"/>
+<label x="400.05" y="125.73" size="1.778" layer="95" rot="R90"/>
+<pinref part="R8" gate="G$1" pin="1"/>
+<wire x1="400.05" y1="142.24" x2="400.05" y2="124.46" width="0.1524" layer="91"/>
+<wire x1="403.86" y1="142.24" x2="400.05" y2="142.24" width="0.1524" layer="91"/>
+<junction x="400.05" y="142.24"/>
 </segment>
 </net>
@@
 <segment>
 <pinref part="2B" gate="G$1" pin="TP"/>
-<wire x1="397.51" y1="143.51" x2="397.51" y2="124.46" width="0.1524" layer="91"/>
-<label x="397.51" y="125.73" size="1.778" layer="95" rot="R90"/>
-</segment>
-</net>
+<wire x1="412.75" y1="143.51" x2="412.75" y2="142.24" width="0.1524" layer="91"/>
+<label x="412.75" y="125.73" size="1.778" layer="95" rot="R90"/>
+<pinref part="R9" gate="G$1" pin="1"/>
+<wire x1="412.75" y1="142.24" x2="412.75" y2="124.46" width="0.1524" layer="91"/>
+<wire x1="416.56" y1="142.24" x2="412.75" y2="142.24" width="0.1524" layer="91"/>
+<junction x="412.75" y="142.24"/>
+</segment>
+</net>
